Commit message: modif rviz

File: urdf/ZumoCarto.urdf (robot description, URDF)
Before this commit: robot ZumoCarto, 4 links, 3 joints
Joints:
- joint joint1: axis 0 0 1 -> (none); child base -> odom; type planar -> floating
- joint jointodom: child odom -> base; parent base -> odom

Commit message: modif rviz3

File: urdf/ZumoCarto.urdf (robot description, URDF)
Before this commit: robot ZumoCarto, 4 links, 3 joints
Joints:
- joint joint1: type floating -> fixed
- joint jointodom: type fixed -> floating

Commit message: ca tourne!!

File: urdf/ZumoCarto.urdf (robot description, URDF)
Before this commit: robot ZumoCarto, 4 links, 3 joints
Links:
- removed link base
- removed link map
- removed link odom
- added link base_link; visual mesh filename=package://ZumoCarto/urdf/zumo.STL scale=0.1 0.1 0.1
- added link scan
Joints:
- removed joint joint1
- removed joint jointodom
- added joint jointscan: type fixed, parent base_link, child scan, origin xyz=0 0 0.08 rpy=0 0 0
- joint jointimu: parent base -> base_link

Commit message: readme maj 2

File: urdf/ZumoCarto.urdf (robot description, URDF)
Before this commit: robot ZumoCarto, 3 links, 2 joints
Links:
- link base_link: geometry visual mesh filename=package://ZumoCarto/urdf/zumo.STL scale=1 1 1
